File: controller/plotter_board.kicad_pcb (KiCad board)
At the start: 2 copper layers, 100.1 x 100.1 mm, 89 parts, among them IC1 TMC2208, IC2 TMC2208, J1 Extenal_power, J10 PSU, J2 USB_Serial, J3 SD_Card, J4 OLED, J5 LEDS, J6 Stepper_ribbon, J7 Control_buttons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

Commit message: Upload files
Parts:
- moved R19 0.10 mm to (119.5, 99.5)
Connections:
- IC1 pad 29: (no net) -> GND
Routing:
- net SCL: track 46.4 -> 43.1 mm, vias 3 -> 2
- net GND: track 39.0 -> 37.8 mm, vias 441 -> 442
- net +3V3: track 264.0 -> 263.0 mm
Other:
- board text added: "LONG AXIS LIMIT 15 LONG AXIS STEP 26 LONG AXIS DIR 25 SHORT AXIS LIMIT 13 SHORT AXIS STEP 12 SHORT AXIS DIR 14 STEPPER ENABLE 27 SOLENOID 2 PAPER HOLD BUTT 36 SHIFT REGISTER INT 34 PAUSE LED 4 POWER LED 17 E-BED 16"
- board text removed: "LONG AXIS LIMIT 15 LONG AXIS STEP 26 LONG AXIS DIR 25 SHORT AXIS LIMIT 13 SHORT AXIS STEP 12 SHORT AXIS DIR 14 STEPPER ENABLE 27 SOLENOID 2 PAPER HOLD BUTT 36 SHIFT REGISTER INT 34 PAUSE LED 26 POWER LED 17 E-BED 16"
