File: controller/plotter_board.sch (KiCad schematic (older format))
At the start: 85 parts, among them IC1 TMC2208, IC2 TMC2208, J1 Extenal_power, J10 PSU, J2 USB_Serial, J3 SD_Card, J4 OLED, J5 LEDS, J6 Stepper_ribbon, J7 Control_buttons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

Commit message: Fix pin maps
Parts:
- removed D6: LED_BLUE, LED_SMD:LED_0603_1608Metric, symbol Device:LED
- removed R14: 2K2, Resistor_SMD:R_0603_1608Metric, symbol Device:R
Connections:
- net PAPER_HOLD: now also U1.5 (SENSOR_VN); no longer U1.24 (IO2)
- net PWM_SOLENOID: now also U1.24 (IO2); no longer U1.9 (IO33)
- no-connect marks 24 -> 23
Other:
- moved on the sheet: JP1, R9
Changed lines of the file:
@@
 Text GLabel 3550 7250 2    50   Input ~ 0
 SCL
-Text GLabel 3550 5950 2    50   Input ~ 0
+Text GLabel 2350 6050 0    50   Input ~ 0
 PAPER_HOLD
 Text GLabel 2350 7700 0    50   Input ~ 0
@@
 Wire Wire Line
 	7625 6725 7625 6775
-Text GLabel 3550 7850 2    50   Input ~ 0
+Text GLabel 3550 5950 2    50   Input ~ 0
 PWM_SOLENOID
 Text GLabel 7475 6725 0    50   Input ~ 0
@@
 Text GLabel 3550 6450 2    50   Input ~ 0
 SHORT_AXIS_LIMIT_O
-$Comp
-L Device:LED D6
-U 1 1 61AEC6E5
-P 6875 7925
-F 0 "D6" V 6875 8050 50  0000 C CNN
-F 1 "LED_BLUE" V 6775 8150 50  0000 C CNN
-F 2 "LED_SMD:LED_0603_1608Metric" H 6875 7925 50  0001 C CNN
-F 3 "~" H 6875 7925 50  0001 C CNN
-F 4 "C72041" H 6875 7925 50  0001 C CNN "LCSC"
-	1    6875 7925
-	0    -1   -1   0
-$EndComp
-$Comp
-L Device:R R14
-U 1 1 61BA9820
-P 6875 7625
-F 0 "R14" H 7025 7625 50  0000 C CNN
-F 1 "2K2" V 6875 7625 50  0000 C CNN
-F 2 "Resistor_SMD:R_0603_1608Metric" V 6805 7625 50  0001 C CNN
-F 3 "~" H 6875 7625 50  0001 C CNN
-F 4 "C4190" V 6875 7625 50  0001 C CNN "LCSC"
-	1    6875 7625
-	-1   0    0    1
-$EndComp
 Wire Wire Line
 	13125 7550 13125 7750
@@
 $EndComp
 Wire Wire Line
-	6750 7475 6875 7475
-Connection ~ 6875 7475
-Wire Wire Line
-	6875 7475 7125 7475
-Wire Wire Line
-	6875 8075 7525 8075
-Wire Wire Line
 	7525 8075 7525 7775
-Connection ~ 7525 8075
 Wire Wire Line
 	7025 9650 7025 9750
@@
 L Device:R R9
 U 1 1 61B16CBF
-P 4475 5950
-F 0 "R9" V 4575 5950 50  0000 C CNN
-F 1 "22K" V 4475 5950 50  0000 C CNN
-F 2 "Resistor_SMD:R_0402_1005Metric" V 4405 5950 50  0001 C CNN
-F 3 "~" H 4475 5950 50  0001 C CNN
-F 4 "C25768" V 4475 5950 50  0001 C CNN "LCSC"
-	1    4475 5950
-	0    1    1    0
+P 1575 6050
+F 0 "R9" V 1675 6050 50  0000 C CNN
+F 1 "22K" V 1575 6050 50  0000 C CNN
+F 2 "Resistor_SMD:R_0402_1005Metric" V 1505 6050 50  0001 C CNN
+F 3 "~" H 1575 6050 50  0001 C CNN
+F 4 "C25768" V 1575 6050 50  0001 C CNN "LCSC"
+	1    1575 6050
+	0    -1   -1   0
 $EndComp
 $Comp
 L Device:Jumper_NO_Small JP1
 U 1 1 61B17BB4
-P 4875 5950
-F 0 "JP1" H 4875 6025 50  0000 C CNN
-F 1 "TEST_JUMPER" H 4875 5850 50  0000 C CNN
-F 2 "Jumper:SolderJumper-2_P1.3mm_Open_RoundedPad1.0x1.5mm" H 4875 5950 50  0001 C CNN
-F 3 "~" H 4875 5950 50  0001 C CNN
-	1    4875 5950
-	1    0    0    -1
+P 1175 6050
+F 0 "JP1" H 1175 6125 50  0000 C CNN
+F 1 "TEST_JUMPER" H 1125 5950 50  0000 C CNN
+F 2 "Jumper:SolderJumper-2_P1.3mm_Open_RoundedPad1.0x1.5mm" H 1175 6050 50  0001 C CNN
+F 3 "~" H 1175 6050 50  0001 C CNN
+	1    1175 6050
+	-1   0    0    1
 $EndComp
 $Comp
 L power:+3V3 #PWR09
 U 1 1 61B183AE
-P 5125 5950
-F 0 "#PWR09" H 5125 5800 50  0001 C CNN
-F 1 "+3V3" H 5140 6123 50  0000 C CNN
-F 2 "" H 5125 5950 50  0001 C CNN
-F 3 "" H 5125 5950 50  0001 C CNN
-	1    5125 5950
-	1    0    0    -1
-$EndComp
-Wire Wire Line
-	5125 5950 4975 5950
-Wire Wire Line
-	4775 5950 4625 5950
-Wire Wire Line
-	4325 5950 3550 5950
+P 925 6050
+F 0 "#PWR09" H 925 5900 50  0001 C CNN
+F 1 "+3V3" H 940 6223 50  0000 C CNN
+F 2 "" H 925 6050 50  0001 C CNN
+F 3 "" H 925 6050 50  0001 C CNN
+	1    925  6050
+	1    0    0    -1
+$EndComp
+Wire Wire Line
+	925  6050 1075 6050
+Wire Wire Line
+	1275 6050 1425 6050
 Wire Wire Line
 	7300 1900 7300 1950
@@
 $EndComp
 NoConn ~ 2350 5950
-NoConn ~ 2350 6050
 NoConn ~ 3550 7750
 NoConn ~ 3550 8050
+Wire Wire Line
+	1725 6050 2350 6050
+Wire Wire Line
+	6750 7475 7125 7475
 $EndSCHEMATC

Commit message: Upload files
Parts:
- IC1, IC2: symbol plotter_board-rescue:TMC2208-SilentStepStick-TMC2208_v11-eagle-import -> plotter_board-rescue:TMC2208-SilentStepStick-TMC2208_v11-eagle-import-plotter_board-rescue-plotter_board-rescue
- R12, R13, R28, R29: symbol plotter_board-rescue:R-EU_M0805-SilentStepStick-TMC2208_v11-eagle-import -> plotter_board-rescue:R-EU_M0805-SilentStepStick-TMC2208_v11-eagle-import-plotter_board-rescue-plotter_board-rescue
- R20, R5: symbol plotter_board-rescue:RESISTOR-0402-SilentStepStick-TMC2208_v11-eagle-import -> plotter_board-rescue:RESISTOR-0402-SilentStepStick-TMC2208_v11-eagle-import-plotter_board-rescue-plotter_board-rescue
Changed lines of the file:
@@
 	4300 1950 4205 1950
 $Comp
-L plotter_board-rescue:TMC2208-SilentStepStick-TMC2208_v11-eagle-import IC1
+L plotter_board-rescue:TMC2208-SilentStepStick-TMC2208_v11-eagle-import-plotter_board-rescue-plotter_board-rescue IC1
 U 1 1 22F7723E
 P 5100 2950
@@
 $EndComp
 $Comp
-L plotter_board-rescue:R-EU_M0805-SilentStepStick-TMC2208_v11-eagle-import R12
+L plotter_board-rescue:R-EU_M0805-SilentStepStick-TMC2208_v11-eagle-import-plotter_board-rescue-plotter_board-rescue R12
 U 1 1 0DC3F8C1
 P 6150 4350
@@
 	9550 2500 9550 2550
 $Comp
-L plotter_board-rescue:RESISTOR-0402-SilentStepStick-TMC2208_v11-eagle-import R20
+L plotter_board-rescue:RESISTOR-0402-SilentStepStick-TMC2208_v11-eagle-import-plotter_board-rescue-plotter_board-rescue R20
 U 1 1 60E92562
 P 9550 2300
@@
 $EndComp
 $Comp
-L plotter_board-rescue:R-EU_M0805-SilentStepStick-TMC2208_v11-eagle-import R29
+L plotter_board-rescue:R-EU_M0805-SilentStepStick-TMC2208_v11-eagle-import-plotter_board-rescue-plotter_board-rescue R29
 U 1 1 60E92600
 P 11950 4350
@@
 $EndComp
 $Comp
-L plotter_board-rescue:R-EU_M0805-SilentStepStick-TMC2208_v11-eagle-import R28
+L plotter_board-rescue:R-EU_M0805-SilentStepStick-TMC2208_v11-eagle-import-plotter_board-rescue-plotter_board-rescue R28
 U 1 1 60E9260B
 P 11600 4350
@@
 	11350 1950 11550 1950
 $Comp
-L plotter_board-rescue:TMC2208-SilentStepStick-TMC2208_v11-eagle-import IC2
+L plotter_board-rescue:TMC2208-SilentStepStick-TMC2208_v11-eagle-import-plotter_board-rescue-plotter_board-rescue IC2
 U 1 1 60E9253D
 P 10550 2950
@@
 	4205 2550 4300 2550
 $Comp
-L plotter_board-rescue:RESISTOR-0402-SilentStepStick-TMC2208_v11-eagle-import R5
+L plotter_board-rescue:RESISTOR-0402-SilentStepStick-TMC2208_v11-eagle-import-plotter_board-rescue-plotter_board-rescue R5
 U 1 1 60EA6620
 P 4205 2310
@@
 	12725 1950 13100 1950
 $Comp
-L plotter_board-rescue:R-EU_M0805-SilentStepStick-TMC2208_v11-eagle-import R13
+L plotter_board-rescue:R-EU_M0805-SilentStepStick-TMC2208_v11-eagle-import-plotter_board-rescue-plotter_board-rescue R13
 U 1 1 F05E0EDF
 P 6500 4350
