File: controller/plotter_board.sch (KiCad schematic (older format))
At the start: 83 parts, among them IC1 TMC2208, IC2 TMC2208, J1 Extenal_power, J10 PSU, J2 USB_Serial, J3 SD_Card, J4 OLED, J5 LEDS, J6 Stepper_ribbon, J7 Control_buttons, J8 Stepper_short, J9 Pen_Buttons, Q1 AO3400A, Q2 2N7002, Q3 2N7002, Q4 AO3401A, Q5 AO3401A, U1 ESP32-WROOM, U2 PCA9539PW, U3 AZ1117-3.3

Commit message: Upload files
Parts:
- removed R19, R3: 10K, Resistor_SMD:R_0402_1005Metric, symbol Device:R
- added D6: LED_BLUE, LED_SMD:LED_0603_1608Metric, symbol Device:LED
- added H5, H6, H7: MountingHole, MountingHole:MountingHole_3.7mm_Pad_Via, symbol Mechanical:MountingHole
- added R14: 2K2, Resistor_SMD:R_0603_1608Metric, symbol Device:R
- added R9: 4K7, Resistor_SMD:R_0402_1005Metric, symbol Device:R
- IC1, IC2: value TMC2208 -> TMC2209
- renumbered D3 to D2, D2 to D3, D5 to D4, D4 to D5, R20 to R19, R21 to R20, R22 to R21, R23 to R22, R24 to R23, R25 to R24, R26 to R25, R27 to R26, R28 to R27, R29 to R28, R4 to R3, R5 to R4, R8 to R5, R7 to R6, R6 to R7, R9 to R8
Connections:
- net +3V3: no longer IC2.10 (MS2)
- net GND: now also IC2.10 (MS2), D6.1 (K)
- net LONG_AXIS_LIMIT_O: now also U1.4 (SENSOR_VP); no longer U1.23 (IO15)
- net PWM_SOLENOID: now also R14.2
- net SHORT_AXIS_LIMIT_O: now also U1.7 (IO35); no longer U1.16 (IO13)
- net SHORT_DIAG: now reaches IC1.11 (DIAG)
- net SHORT_DIAG: now also U1.16 (IO13)
- net TMC_UART: now reaches IC1.14 (PDN_UART)
- net TMC_UART: now also IC2.14 (PDN_UART), U1.9 (IO33), R9.2
- net LONG_DIAG: now reaches IC2.11 (DIAG)
- net LONG_DIAG: now also U1.23 (IO15)
- net TMC_UART_RX: now reaches U1.8 (IO32)
- net TMC_UART_RX: now also R9.1
- new net: D6.2 (A), R14.1
- no-connect marks 23 -> 18
Other:
- moved on the sheet: C14, C17, C18, C19, D4, D5, JP1, R10, R5, R6, R7, R8
