File: Daugter_board/Daugter_board.kicad_pcb (KiCad board)
At the start: 2 copper layers, 41.7 x 34.8 mm, 19 parts, among them J1 USB_C_Receptacle_USB2.0, J2 Micro_SD_Card, J3 USB_Serial, J4 SD_Card, Q1 MMBT3904, Q2 MMBT3904, U1 AP1117-33, U2 CH340B

Commit message: Upload files
Parts:
- J1: footprint Connector_USB:USB_C_Receptacle_HRO_TYPE-C-31-M-12 -> plotter_board:USB_C_Receptacle_HRO_TYPE-C-31-M-12
